File: schematics/RAM-ROM.sch (KiCad schematic (older format))
At the start: 2 parts, among them U4 2764, U5 SIMM16M

Commit message: merge from Jani's commit
Changed lines of the file:
@@
 Wire Wire Line
 	1700 700  1300 700
-Connection ~ 1300 700
 Wire Bus Line
 	2550 950  2550 1800
@@
 Wire Bus Line
 	7000 1600 7000 2900
-Wire Bus Line
-	950  1100 950  2300
 $EndSCHEMATC
