File: schematics/RAM-ROM.sch (KiCad schematic (older format))
At the start: 2 parts, among them U4 2764, U5 SIMM16M

Commit message: add bus labels, hierarchial labels
Parts:
- added C? (x2): 0.1uF, symbol Device:C
Connections:
- net labels added: A0, A1, A10, A11, A12, A2, A3, A4, A5, A6, A7, A8, A9, D0, D1, D2, D3, D4, D5, D6, D7, DQ0, DQ1, DQ2, DQ3, DQ4, DQ5, DQ6, DQ7, DQ[0..7], MA0, MA1, MA10, MA11, MA2, MA3, MA4, MA5, MA6, MA7, MA8, MA9, VCC
- net labels removed: DQ[0..8], Vcc
- wire segments 30 -> 66
Other:
- moved on the sheet: U5

Commit message: begin wiring up the hierarchial sheets
Connections:
- net labels added: R~W
- net labels removed: RW
Changed lines of the file:
@@
 $Descr A4 11693 8268
 encoding utf-8
-Sheet 6 7
+Sheet 7 7
 Title ""
 Date ""
@@
 Wire Wire Line
 	7300 3650 7500 3650
-Text GLabel 6600 3200 0    50   Input ~ 10
-ROM_EN
 Wire Wire Line
 	7100 3200 6600 3200
@@
 Entry Wire Line
 	2500 3000 2600 2900
-Text GLabel 2200 3300 0    50   Input ~ 10
-RW
-Text GLabel 2200 3150 0    50   Input ~ 10
-RAS
-Text GLabel 2200 3000 0    50   Input ~ 10
-CAS
 Wire Wire Line
 	2300 3200 2300 3150
@@
 Wire Bus Line
 	2500 1750 2500 3000
+Text HLabel 2200 3000 0    50   Input ~ 0
+CAS
+Text HLabel 2200 3150 0    50   Input ~ 0
+RAS
+Text HLabel 2200 3300 0    50   Input ~ 0
+R~W
+Text HLabel 6600 3200 0    50   Input ~ 0
+ROM_EN
 $EndSCHEMATC

Commit message: Add SIMM size select jumpers
Parts:
- added JP? (x3): Jumper_2_Open, symbol Jumper:Jumper_2_Open
Connections:
- wire segments 66 -> 67
Changed lines of the file:
@@
 Entry Wire Line
 	2500 2700 2600 2600
-Entry Wire Line
-	2500 2800 2600 2700
-Entry Wire Line
-	2500 2900 2600 2800
-Entry Wire Line
-	2500 3000 2600 2900
 Wire Wire Line
 	2300 3200 2300 3150
@@
 Text HLabel 6750 1600 0    50   Input ~ 0
 A[0..15]
-Text GLabel 5500 4300 2    50   Output ~ 10
+Text GLabel 9300 5700 2    50   Output ~ 10
 VCC
-Text GLabel 5500 4600 2    50   Output ~ 10
+Text GLabel 9300 6000 2    50   Output ~ 10
 GND
 $Comp
 L Device:C C?
 U 1 1 616CE492
-P 4450 4450
-F 0 "C?" H 4565 4496 50  0000 L CNN
-F 1 "0.1uF" H 4565 4405 50  0000 L CNN
-F 2 "" H 4488 4300 50  0001 C CNN
-F 3 "~" H 4450 4450 50  0001 C CNN
-	1    4450 4450
+P 8250 5850
+F 0 "C?" H 8365 5896 50  0000 L CNN
+F 1 "0.1uF" H 8365 5805 50  0000 L CNN
+F 2 "" H 8288 5700 50  0001 C CNN
+F 3 "~" H 8250 5850 50  0001 C CNN
+	1    8250 5850
 	1    0    0    -1
 $EndComp
@@
 L Device:C C?
 U 1 1 616CE8B0
-P 4950 4450
-F 0 "C?" H 5065 4496 50  0000 L CNN
-F 1 "0.1uF" H 5065 4405 50  0000 L CNN
-F 2 "" H 4988 4300 50  0001 C CNN
-F 3 "~" H 4950 4450 50  0001 C CNN
-	1    4950 4450
-	1    0    0    -1
-$EndComp
-Text HLabel 4100 4300 0    50   Input ~ 0
+P 8750 5850
+F 0 "C?" H 8865 5896 50  0000 L CNN
+F 1 "0.1uF" H 8865 5805 50  0000 L CNN
+F 2 "" H 8788 5700 50  0001 C CNN
+F 3 "~" H 8750 5850 50  0001 C CNN
+	1    8750 5850
+	1    0    0    -1
+$EndComp
+Text HLabel 7900 5700 0    50   Input ~ 0
 VCC
-Text HLabel 4100 4600 0    50   Input ~ 0
+Text HLabel 7900 6000 0    50   Input ~ 0
 GND
 Wire Wire Line
-	4100 4600 4450 4600
-Connection ~ 4450 4600
-Wire Wire Line
-	4450 4600 4950 4600
-Connection ~ 4950 4600
-Wire Wire Line
-	4950 4600 5500 4600
-Wire Wire Line
-	4100 4300 4450 4300
-Connection ~ 4450 4300
-Wire Wire Line
-	4450 4300 4950 4300
-Connection ~ 4950 4300
-Wire Wire Line
-	4950 4300 5500 4300
+	7900 6000 8250 6000
+Connection ~ 8250 6000
+Wire Wire Line
+	8250 6000 8750 6000
+Connection ~ 8750 6000
+Wire Wire Line
+	8750 6000 9300 6000
+Wire Wire Line
+	7900 5700 8250 5700
+Connection ~ 8250 5700
+Wire Wire Line
+	8250 5700 8750 5700
+Connection ~ 8750 5700
+Wire Wire Line
+	8750 5700 9300 5700
 Text Label 6950 1600 0    50   ~ 0
 A0
@@
 Wire Wire Line
 	2600 2600 2800 2600
-Wire Wire Line
-	2600 2700 2800 2700
-Wire Wire Line
-	2600 2800 2800 2800
-Wire Wire Line
-	2600 2900 2800 2900
 Wire Bus Line
 	2500 1750 2450 1750
-Text HLabel 2450 1750 0    50   Input ~ 0
-MA[0..11]
 Text Label 2650 1800 0    50   ~ 0
 MA0
@@
 Text Label 2650 2600 0    50   ~ 0
 MA8
-Text Label 2650 2700 0    50   ~ 0
-MA9
-Text Label 2650 2800 0    50   ~ 0
-MA10
-Text Label 2650 2900 0    50   ~ 0
-MA11
 Wire Wire Line
 	2200 3300 2800 3300
@@
 Wire Wire Line
 	2300 3100 2650 3100
-Wire Bus Line
-	4500 1700 4500 2550
-Wire Bus Line
-	8150 1450 8150 2250
-Wire Bus Line
-	6800 1600 6800 2900
-Wire Bus Line
-	2500 1750 2500 3000
 Text HLabel 2200 3000 0    50   Input ~ 0
 CAS
@@
 Text HLabel 6600 3200 0    50   Input ~ 0
 ROM_EN
+Text GLabel 2800 2700 0    50   Input ~ 0
+MA9
+Text GLabel 2800 2800 0    50   Input ~ 0
+MA10
+Text GLabel 2800 2900 0    50   Input ~ 0
+MA11
+Text HLabel 8050 4950 0    50   Input ~ 0
+MA[0..11]
+Text GLabel 3600 4350 2    50   Output ~ 0
+MA9
+Text GLabel 3600 4700 2    50   Output ~ 0
+MA10
+Text GLabel 3600 5050 2    50   Output ~ 0
+MA11
+$Comp
+L Jumper:Jumper_2_Open JP?
+U 1 1 61A2D8CC
+P 3400 4350
+F 0 "JP?" H 3400 4585 50  0000 C CNN
+F 1 "Jumper_2_Open" H 3400 4494 50  0000 C CNN
+F 2 "" H 3400 4350 50  0001 C CNN
+F 3 "~" H 3400 4350 50  0001 C CNN
+	1    3400 4350
+	1    0    0    -1
+$EndComp
+$Comp
+L Jumper:Jumper_2_Open JP?
+U 1 1 61A2FC07
+P 3400 4700
+F 0 "JP?" H 3400 4935 50  0000 C CNN
+F 1 "Jumper_2_Open" H 3400 4844 50  0000 C CNN
+F 2 "" H 3400 4700 50  0001 C CNN
+F 3 "~" H 3400 4700 50  0001 C CNN
+	1    3400 4700
+	1    0    0    -1
+$EndComp
+$Comp
+L Jumper:Jumper_2_Open JP?
+U 1 1 61A300DC
+P 3400 5050
+F 0 "JP?" H 3400 5285 50  0000 C CNN
+F 1 "Jumper_2_Open" H 3400 5194 50  0000 C CNN
+F 2 "" H 3400 5050 50  0001 C CNN
+F 3 "~" H 3400 5050 50  0001 C CNN
+	1    3400 5050
+	1    0    0    -1
+$EndComp
+Wire Wire Line
+	3200 4350 3000 4350
+Wire Wire Line
+	3200 4700 3000 4700
+Wire Wire Line
+	3200 5050 3000 5050
+Entry Wire Line
+	3000 4350 2900 4250
+Entry Wire Line
+	3000 4700 2900 4600
+Entry Wire Line
+	3000 5050 2900 4950
+Wire Bus Line
+	2900 4150 2850 4150
+Wire Wire Line
+	8050 4950 8200 4950
+Wire Bus Line
+	2900 4150 2900 4950
+Wire Bus Line
+	4500 1700 4500 2550
+Wire Bus Line
+	8150 1450 8150 2250
+Wire Bus Line
+	2500 1750 2500 2700
+Wire Bus Line
+	6800 1600 6800 2900
+Text GLabel 8200 4950 2    50   Output ~ 0
+MA[0..11]
+Text GLabel 2850 4150 0    50   Input ~ 0
+MA[0..11]
+Text GLabel 2450 1750 0    50   Input ~ 0
+MA[0..11]
+Text Label 3050 4350 0    50   ~ 0
+MA9
+Text Label 3050 4700 0    50   ~ 0
+MA10
+Text Label 3050 5050 0    50   ~ 0
+MA11
 $EndSCHEMATC

Commit message: Added a few lost power connections and no_connect entries.
Connections:
- wire segments 67 -> 79
Changed lines of the file:
@@
 $Descr A4 11693 8268
 encoding utf-8
-Sheet 7 7
+Sheet 5 7
 Title ""
 Date ""
@@
 	7500 1400 7500 1000
 Wire Wire Line
-	7500 1000 7200 1000
+	7500 1000 7300 1000
 Text GLabel 7200 3650 0    50   Input ~ 10
 GND
@@
 Connection ~ 7300 3650
 Wire Wire Line
-	7300 3650 7500 3650
+	7300 3650 7350 3650
 Wire Wire Line
 	7100 3200 6600 3200
@@
 Wire Wire Line
 	8050 4950 8200 4950
-Wire Bus Line
-	2900 4150 2900 4950
-Wire Bus Line
-	4500 1700 4500 2550
-Wire Bus Line
-	8150 1450 8150 2250
-Wire Bus Line
-	2500 1750 2500 2700
-Wire Bus Line
-	6800 1600 6800 2900
 Text GLabel 8200 4950 2    50   Output ~ 0
 MA[0..11]
@@
 Text Label 3050 5050 0    50   ~ 0
 MA11
+Wire Wire Line
+	3350 3450 3350 3800
+Wire Wire Line
+	3350 3800 3450 3800
+Wire Wire Line
+	7350 3800 7350 3650
+Connection ~ 7350 3650
+Wire Wire Line
+	7350 3650 7500 3650
+Wire Wire Line
+	3450 3450 3450 3800
+Connection ~ 3450 3800
+Wire Wire Line
+	3450 3800 7350 3800
+Wire Wire Line
+	3450 1650 3450 1150
+Wire Wire Line
+	3450 1150 7300 1150
+Wire Wire Line
+	7300 1150 7300 1000
+Connection ~ 7300 1000
+Wire Wire Line
+	7300 1000 7200 1000
+Wire Wire Line
+	3350 1150 3450 1150
+Connection ~ 3450 1150
+Wire Wire Line
+	3350 1150 3350 1650
+Wire Bus Line
+	2900 4150 2900 4950
+Wire Bus Line
+	4500 1700 4500 2550
+Wire Bus Line
+	8150 1450 8150 2250
+Wire Bus Line
+	2500 1750 2500 2700
+Wire Bus Line
+	6800 1600 6800 2900
 $EndSCHEMATC
