File: schematics/audio.sch (KiCad schematic (older format))
At the start: 3 parts, among them J13 Left Audio, J14 Right Audio, U12 EN5503DOC

Commit message: Removed EN5503DOC chip from IO2 sheet as it is now on it's own separate sheet. Changed description texts to reflect the change.
Other:
- note added: "EN5503 DOC Audio + outputs\n64kB Audio DRAM\n"
- note removed: "Audio + outputs\nAudio DRAM\nIDE-Interface\nFloppy drive interface"
Changed lines of the file:
@@
 Text Notes 10600 7650 0    50   ~ 10
 0
-Text Notes 7050 6950 0    50   ~ 10
-Audio + outputs\nAudio DRAM\nIDE-Interface\nFloppy drive interface
+Text Notes 7050 6800 0    50   ~ 10
+EN5503 DOC Audio + outputs\n64kB Audio DRAM\n
 Wire Wire Line
 	11150 3600 11150 550
@@
 AR Path="/5EFB7822" Ref="U12"  Part="1"
 AR Path="/5F47C633/5EFB7822" Ref="U12"  Part="1"
+AR Path="/5F16299B/5EFB7822" Ref="U12"  Part="1"
 F 0 "U12" H 5900 2275 50  0000 C CNN
 F 1 "EN5503DOC" H 5900 2184 50  0000 C CNN

Commit message: finish up hierarchial pins (as they stand now)
Parts:
- added C?: 0.1uF, symbol Device:C
Connections:
- net labels added: VCC
- net labels removed: Vcc
- wire segments 10 -> 14
Changed lines of the file:
@@
 $Descr A4 11693 8268
 encoding utf-8
-Sheet 7 7
+Sheet 5 7
 Title ""
 Date ""
@@
 Wire Wire Line
 	5450 4150 5300 4150
-Text HLabel 5300 3950 0    50   Input ~ 0
+Text HLabel 5300 3950 0    50   Output ~ 0
 ~IRQ
 Text HLabel 5300 4150 0    50   Input ~ 0
@@
 	6350 2350 6500 2350
 Text GLabel 6500 2350 2    50   Input ~ 0
-Vcc
+VCC
+Text GLabel 10050 4650 2    50   Output ~ 0
+GND
+Text GLabel 10050 4350 2    50   Output ~ 0
+VCC
+$Comp
+L Device:C C?
+U 1 1 630269F5
+P 9800 4500
+F 0 "C?" H 9915 4546 50  0000 L CNN
+F 1 "0.1uF" H 9915 4455 50  0000 L CNN
+F 2 "" H 9838 4350 50  0001 C CNN
+F 3 "~" H 9800 4500 50  0001 C CNN
+	1    9800 4500
+	1    0    0    -1
+$EndComp
+Text HLabel 9500 4350 0    50   Input ~ 0
+VCC
+Text HLabel 9500 4650 0    50   Input ~ 0
+GND
+Wire Wire Line
+	9500 4650 9800 4650
+Connection ~ 9800 4650
+Wire Wire Line
+	9800 4650 10050 4650
+Wire Wire Line
+	9500 4350 9800 4350
+Connection ~ 9800 4350
+Wire Wire Line
+	9800 4350 10050 4350
 $EndSCHEMATC
