File: schematics/io-2.sch (KiCad schematic (older format))
At the start: 14 parts, among them J13 FDC Connector, J9 IDE Connector, U11 WD1772, U13 74LS574, U14 74LS574, U15 74LS245, U16 74LS245

Commit message: another note for the future
Other:
- note added: "This is active high! >>>"
Changed lines of the file:
@@
 Wire Bus Line
 	5300 2650 5300 3950
+Text Notes 550  5000 0    50   ~ 0
+This is active high! >>>
 $EndSCHEMATC

Commit message: rename A[0..23] to A[0..15]
Connections:
- net labels removed: A[0..23]
Changed lines of the file:
@@
 	1850 5950 1950 5850
 Text GLabel 1850 5800 0    50   Input ~ 10
-A[0..23]
+A[0..15]
 Wire Wire Line
 	1600 5600 1450 5600
@@
 D6
 Text GLabel 8500 6100 2    50   Output ~ 10
-A[0..23]
+A[0..15]
 Text GLabel 8500 6300 2    50   BiDi ~ 10
 D[0..7]
 Text HLabel 8250 6100 0    50   Input ~ 0
-A[0..23]
+A[0..15]
 Text HLabel 8250 6300 0    50   BiDi ~ 0
 D[0..7]

Commit message: begin wiring up the hierarchial sheets
Changed lines of the file:
@@
 Wire Wire Line
 	9650 2050 9650 1850
-Text GLabel 9500 2950 2    50   Input ~ 0
-IDE_CS0
 Wire Wire Line
 	9500 3050 9350 3050
@@
 Wire Wire Line
 	9000 3350 9350 3350
-Text GLabel 9500 3050 2    50   Input ~ 0
-IDE_CS1
 Wire Wire Line
 	9350 2950 9500 2950
@@
 Text Notes 550  5000 0    50   ~ 0
 This is active high! >>>
+Text HLabel 9500 2950 2    50   Input ~ 0
+IDE_CS0
+Text HLabel 9500 3050 2    50   Input ~ 0
+IDE_CS1
 $EndSCHEMATC

Commit message: additional fixups
Changed lines of the file:
@@
 $Descr A4 11693 8268
 encoding utf-8
-Sheet 4 7
+Sheet 3 7
 Title ""
 Date ""
@@
 Wire Wire Line
 	4950 5250 4300 5250
-Text GLabel 4150 5450 0    50   Input ~ 0
-FDC_DSKCHG
 Wire Wire Line
 	4150 5350 4250 5350
@@
 Wire Wire Line
 	5550 5550 5550 5000
-Text GLabel 4150 5350 0    50   Input ~ 0
-FDC_DRVA
 Wire Wire Line
 	4200 5100 4200 5250
@@
 Wire Wire Line
 	5450 5350 5500 5350
-Text GLabel 4150 5250 0    50   Input ~ 0
-FDC_MTREN
 Wire Wire Line
 	4700 5150 4150 5150
@@
 Wire Wire Line
 	4950 5450 4700 5450
-Text GLabel 4150 5150 0    50   Input ~ 0
-FDC_SIDE
 Wire Wire Line
 	2600 6950 2950 6950
@@
 Text HLabel 1550 5050 0    50   Output ~ 0
 IRQ_HIGH
-Wire Wire Line
-	8350 2850 8850 2850
-Wire Wire Line
-	8350 2650 8850 2650
-Wire Wire Line
-	8350 2450 8850 2450
-Wire Wire Line
-	8350 2250 8850 2250
-Wire Wire Line
-	8350 2050 8850 2050
-Wire Wire Line
-	8350 1850 8850 1850
-Wire Wire Line
-	8350 1650 8850 1650
-Wire Bus Line
-	9650 2450 9650 2800
-Wire Bus Line
-	1850 5700 1850 5900
-Wire Bus Line
-	1850 5950 1850 6650
-Wire Bus Line
-	2300 950  2300 1950
-Wire Bus Line
-	1800 2650 1800 3950
-Wire Bus Line
-	8250 1450 8250 3100
-Wire Bus Line
-	8400 1350 8400 3000
-Wire Bus Line
-	3950 1050 3950 2450
-Wire Bus Line
-	3550 2450 3550 3550
-Wire Bus Line
-	5700 1050 5700 1950
-Wire Bus Line
-	5300 2650 5300 3950
 Text Notes 550  5000 0    50   ~ 0
 This is active high! >>>
@@
 Text HLabel 9500 3050 2    50   Input ~ 0
 IDE_CS1
+Text HLabel 4150 5150 0    50   Input ~ 0
+FDC_SIDE
+Text HLabel 4150 5250 0    50   Output ~ 0
+FDC_MTREN
+Text HLabel 4150 5350 0    50   Input ~ 0
+FDC_DRVA
+Text HLabel 4150 5450 0    50   Output ~ 0
+FDC_DSKCHG
+Wire Wire Line
+	8350 2850 8850 2850
+Wire Wire Line
+	8350 2650 8850 2650
+Wire Wire Line
+	8350 2450 8850 2450
+Wire Wire Line
+	8350 2250 8850 2250
+Wire Wire Line
+	8350 2050 8850 2050
+Wire Wire Line
+	8350 1850 8850 1850
+Wire Wire Line
+	8350 1650 8850 1650
+Wire Bus Line
+	9650 2450 9650 2800
+Wire Bus Line
+	1850 5700 1850 5900
+Wire Bus Line
+	1850 5950 1850 6650
+Wire Bus Line
+	2300 950  2300 1950
+Wire Bus Line
+	1800 2650 1800 3950
+Wire Bus Line
+	8250 1450 8250 3100
+Wire Bus Line
+	8400 1350 8400 3000
+Wire Bus Line
+	3950 1050 3950 2450
+Wire Bus Line
+	3550 2450 3550 3550
+Wire Bus Line
+	5700 1050 5700 1950
+Wire Bus Line
+	5300 2650 5300 3950
 $EndSCHEMATC
