File: schematics/io-1.sch (KiCad schematic (older format))
At the start: 11 parts, among them J3 Centronics, J4 ps/2 keyb, J5 Joy1, J6 Joy2, J7 rs232, J8 Expansion, U6 wdc65c22, U7 wdc65c22, U8 wdc65c51, U9 MAX233CPP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

Commit message: Fixes to FDC signal mapping.
Connections:
- net GND: now also J7.5, J7.7, U8.1 (VSS), U8.3 (~CS1), U8.8 (~RTS), U9.6 (GND), U9.9 (GND), X3.7 (GND)
- net FDC_SIDE: now reaches U6.10 (PB0)
- net FDC_MTREN: now reaches U6.11 (PB1)
- net FDC_DRVA: now reaches U6.12 (PB2)
- no-connect marks 31 -> 28
Changed lines of the file:
@@
 NoConn ~ 1100 4750
 NoConn ~ 1100 4950
-NoConn ~ 3000 2950
-NoConn ~ 3000 3050
-NoConn ~ 3000 3150
 NoConn ~ 3000 3250
 NoConn ~ 3000 3550
@@
 	1    0    0    -1
 $EndComp
-Wire Wire Line
-	1000 4050 850  4050
 Wire Wire Line
 	850  4050 850  5200
@@
 Wire Wire Line
 	5750 2250 5300 2250
+Wire Wire Line
+	850  4050 1050 4050
+Connection ~ 1050 4050
+Text GLabel 2800 2950 0    50   Input ~ 0
+FDC_SIDE
+Text GLabel 2850 3050 0    50   Input ~ 0
+FDC_MTREN
+Text GLabel 2800 3150 0    50   Input ~ 0
+FDC_DRVA
+Wire Wire Line
+	2800 2950 3000 2950
+Wire Wire Line
+	2850 3050 3000 3050
+Wire Wire Line
+	2800 3150 3000 3150
 Wire Bus Line
 	3350 6850 3350 7100

Commit message: Added support for Diskchange for FDC interface.
Connections:
- net FDC_DSKCHG: now reaches U6.13 (PB3)
- no-connect marks 28 -> 27
Changed lines of the file:
@@
 VIA 1 : Centronics, ps/2\nVIA 2: Joysticks, Expansion\nUART + MAX233 RS232 serialport
-$Comp
-L 65xx:wdc65c22 U6
-U 1 1 5F26FA50
-P 3250 1950
-F 0 "U6" H 3325 2075 50  0000 C CNN
-F 1 "wdc65c22" H 3325 1984 50  0000 C CNN
-F 2 "Package_DIP:DIP-40_W25.4mm" H 3300 1950 50  0001 C CNN
-F 3 "" H 3300 1950 50  0001 C CNN
-	1    3250 1950
-	1    0    0    -1
-$EndComp
 $Comp
 L 65xx:wdc65c22 U7
@@
 NoConn ~ 1100 4750
 NoConn ~ 1100 4950
-NoConn ~ 3000 3250
 NoConn ~ 3000 3550
 NoConn ~ 3000 3650
@@
 Wire Wire Line
 	2800 3150 3000 3150
+$Comp
+L 65xx:wdc65c22 U6
+U 1 1 5F26FA50
+P 3250 1950
+F 0 "U6" H 3325 2075 50  0000 C CNN
+F 1 "wdc65c22" H 3325 1984 50  0000 C CNN
+F 2 "Package_DIP:DIP-40_W25.4mm" H 3300 1950 50  0001 C CNN
+F 3 "" H 3300 1950 50  0001 C CNN
+	1    3250 1950
+	1    0    0    -1
+$EndComp
+Text GLabel 2900 3250 0    50   Input ~ 0
+FDC_DSKCHG
+Wire Wire Line
+	3000 3250 2900 3250
 Wire Bus Line
 	3350 6850 3350 7100

Commit message: finish up hierarchial pins (as they stand now)
Parts:
- added C? (x4): C, symbol Device:C
Connections:
- net labels added: A0, A1, A2, A3, D0, D1, D2, D3, D4, D5, D6, D7, FDC_WTREN
- net labels removed: FDC_MTREN
- wire segments 355 -> 403

Commit message: additional fixups
Changed lines of the file:
@@
 $Descr A4 11693 8268
 encoding utf-8
-Sheet 3 7
+Sheet 6 7
 Title ""
 Date ""
@@
 Text HLabel 2850 3050 0    50   Input ~ 0
 FDC_WTREN
-Text HLabel 2900 3250 0    50   Output ~ 0
+Text HLabel 2900 3250 0    50   Input ~ 0
 FDC_DSKCHG
-Text HLabel 2800 3150 0    50   Input ~ 0
+Text HLabel 2800 3150 0    50   Output ~ 0
 FDC_DRVA
 Text HLabel 6800 700  0    50   Input ~ 0
@@
 Text Label 3300 6950 0    50   ~ 0
 A1
+Text HLabel 2950 5750 0    50   Input ~ 0
+UART_EN
 Wire Bus Line
 	3150 6850 3150 7100
@@
 Wire Bus Line
 	3950 2650 3950 3400
-Text HLabel 2950 5750 0    50   Input ~ 0
-UART_EN
 $EndSCHEMATC

Commit message: Added a few lost power connections and no_connect entries.
Connections:
- no-connect marks 27 -> 28
Changed lines of the file:
@@
 Text HLabel 2950 5750 0    50   Input ~ 0
 UART_EN
+NoConn ~ 3450 6250
 Wire Bus Line
 	3150 6850 3150 7100
