File: schematics/MARCy.kicad_sch (KiCad schematic)
At the start: 5 parts, among them J16 DIN41612_02x32_AB, J17 DIN41612_02x32_AB, J4 JTAG, U8 XC9572XL-TQ100

Commit message: Small tweaks here and there. Added a lot of missing footprint definitions.
Parts:
- C8: footprint (none) -> Capacitor_THT:CP_Radial_D4.0mm_P1.50mm
Changed lines of the file:
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@@
 	(label "A9"
 		(at 135.89 74.93 0)
-		(fields_autoplaced yes)
 		(effects
 			(font
@@
 	(label "A6"
 		(at 135.89 67.31 0)
-		(fields_autoplaced yes)
 		(effects
 			(font
@@
 	(label "A14"
 		(at 135.89 87.63 0)
-		(fields_autoplaced yes)
 		(effects
 			(font
@@
 	(label "A13"
 		(at 135.89 85.09 0)
-		(fields_autoplaced yes)
 		(effects
 			(font
@@
 	(label "A1"
 		(at 135.89 54.61 0)
-		(fields_autoplaced yes)
 		(effects
 			(font
@@
 	(label "A3"
 		(at 135.89 59.69 0)
-		(fields_autoplaced yes)
 		(effects
 			(font
@@
 	(label "A0"
 		(at 135.89 52.07 0)
-		(fields_autoplaced yes)
 		(effects
 			(font
@@
 	(label "A11"
 		(at 135.89 80.01 0)
-		(fields_autoplaced yes)
 		(effects
 			(font
@@
 	(label "A5"
 		(at 135.89 64.77 0)
-		(fields_autoplaced yes)
 		(effects
 			(font
@@
 	(label "A7"
 		(at 135.89 69.85 0)
-		(fields_autoplaced yes)
 		(effects
 			(font
@@
 	(label "A4"
 		(at 135.89 62.23 0)
-		(fields_autoplaced yes)
 		(effects
 			(font
@@
 	(label "A2"
 		(at 135.89 57.15 0)
-		(fields_autoplaced yes)
 		(effects
 			(font
@@
 	(label "A8"
 		(at 135.89 72.39 0)
-		(fields_autoplaced yes)
 		(effects
 			(font
@@
 	(label "A15"
 		(at 135.89 90.17 0)
-		(fields_autoplaced yes)
 		(effects
 			(font
@@
 	(label "A12"
 		(at 135.89 82.55 0)
-		(fields_autoplaced yes)
 		(effects
 			(font
@@
 	(label "A10"
 		(at 135.89 77.47 0)
-		(fields_autoplaced yes)
 		(effects
 			(font
@@
 		(shape output)
 		(at 58.42 86.36 180)
-		(fields_autoplaced yes)
 		(effects
 			(font
@@
 		(shape output)
 		(at 58.42 124.46 180)
-		(fields_autoplaced yes)
 		(effects
 			(font
@@
 		(shape output)
 		(at 58.42 74.93 180)
-		(fields_autoplaced yes)
 		(effects
 			(font
@@
 		(shape input)
 		(at 27.94 180.34 180)
-		(fields_autoplaced yes)
 		(effects
 			(font
@@
 		(shape output)
 		(at 58.42 101.6 180)
-		(fields_autoplaced yes)
 		(effects
 			(font
@@
 		(shape input)
 		(at 58.42 135.89 180)
-		(fields_autoplaced yes)
 		(effects
 			(font
@@
 		(shape output)
 		(at 58.42 82.55 180)
-		(fields_autoplaced yes)
 		(effects
 			(font
@@
 		(shape input)
 		(at 27.94 172.72 180)
-		(fields_autoplaced yes)
 		(effects
 			(font
@@
 		(shape output)
 		(at 58.42 120.65 180)
-		(fields_autoplaced yes)
 		(effects
 			(font
@@
 		(shape output)
 		(at 58.42 71.12 180)
-		(fields_autoplaced yes)
 		(effects
 			(font
@@
 		(shape output)
 		(at 58.42 132.08 180)
-		(fields_autoplaced yes)
 		(effects
 			(font
@@
 		(shape output)
 		(at 58.42 105.41 180)
-		(fields_autoplaced yes)
 		(effects
 			(font
@@
 		(shape output)
 		(at 58.42 128.27 180)
-		(fields_autoplaced yes)
 		(effects
 			(font
@@
 		(shape output)
 		(at 58.42 90.17 180)
-		(fields_autoplaced yes)
 		(effects
 			(font
@@
 		(shape output)
 		(at 58.42 63.5 180)
-		(fields_autoplaced yes)
 		(effects
 			(font
@@
 		(shape output)
 		(at 58.42 93.98 180)
-		(fields_autoplaced yes)
 		(effects
 			(font
@@
 		(shape output)
 		(at 58.42 78.74 180)
-		(fields_autoplaced yes)
 		(effects
 			(font
@@
 		(shape output)
 		(at 58.42 113.03 180)
-		(fields_autoplaced yes)
 		(effects
 			(font
@@
 		(shape output)
 		(at 58.42 116.84 180)
-		(fields_autoplaced yes)
 		(effects
 			(font
@@
 		(shape output)
 		(at 58.42 59.69 180)
-		(fields_autoplaced yes)
 		(effects
 			(font
@@
 		(shape output)
 		(at 58.42 55.88 180)
-		(fields_autoplaced yes)
 		(effects
 			(font
@@
 		(shape output)
 		(at 58.42 52.07 180)
-		(fields_autoplaced yes)
 		(effects
 			(font
@@
 		(shape input)
 		(at 58.42 97.79 180)
-		(fields_autoplaced yes)
 		(effects
 			(font
@@
 		(shape input)
 		(at 144.78 49.53 0)
-		(fields_autoplaced yes)
 		(effects
 			(font
@@
 		(shape output)
 		(at 58.42 109.22 180)
-		(fields_autoplaced yes)
 		(effects
 			(font
@@
 		(shape output)
 		(at 143.51 97.79 0)
-		(fields_autoplaced yes)
 		(effects
 			(font
@@
 			)
 		)
-		(property "Footprint" ""
+		(property "Footprint" "Capacitor_THT:CP_Radial_D4.0mm_P1.50mm"
 			(at 36.5252 180.34 0)
 			(effects
