File: schematics/io-1.kicad_sch (KiCad schematic)
At the start: 15 parts, among them J10 Centronics, J11 ps/2 keyb, J12 Expansion, J13 Joy1, J14 Joy2, J15 rs232, U13 wdc65c22, U14 wdc65c51, U15 MAX233CPP, U16 wdc65c22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

Commit message: Small tweaks here and there. Added a lot of missing footprint definitions.
Parts:
- C13, C14, C15, C16: footprint (none) -> Capacitor_THT:CP_Radial_D4.0mm_P1.50mm
Changed lines of the file:
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@@
 	(label "D5"
 		(at 93.98 82.55 0)
-		(fields_autoplaced yes)
 		(effects
 			(font
@@
 	(label "D3"
 		(at 179.07 77.47 0)
-		(fields_autoplaced yes)
 		(effects
 			(font
@@
 	(label "A3"
 		(at 93.98 64.77 0)
-		(fields_autoplaced yes)
 		(effects
 			(font
@@
 	(label "D1"
 		(at 93.98 72.39 0)
-		(fields_autoplaced yes)
 		(effects
 			(font
@@
 	(label "D6"
 		(at 93.98 85.09 0)
-		(fields_autoplaced yes)
 		(effects
 			(font
@@
 	(label "D3"
 		(at 105.41 158.75 0)
-		(fields_autoplaced yes)
 		(effects
 			(font
@@
 	(label "D7"
 		(at 105.41 168.91 0)
-		(fields_autoplaced yes)
 		(effects
 			(font
@@
 	(label "A1"
 		(at 179.07 59.69 0)
-		(fields_autoplaced yes)
 		(effects
 			(font
@@
 	(label "D4"
 		(at 179.07 80.01 0)
-		(fields_autoplaced yes)
 		(effects
 			(font
@@
 	(label "D0"
 		(at 179.07 69.85 0)
-		(fields_autoplaced yes)
 		(effects
 			(font
@@
 	(label "A0"
 		(at 83.82 173.99 0)
-		(fields_autoplaced yes)
 		(effects
 			(font
@@
 	(label "A1"
 		(at 93.98 59.69 0)
-		(fields_autoplaced yes)
 		(effects
 			(font
@@
 	(label "D6"
 		(at 105.41 166.37 0)
-		(fields_autoplaced yes)
 		(effects
 			(font
@@
 	(label "A0"
 		(at 93.98 57.15 0)
-		(fields_autoplaced yes)
 		(effects
 			(font
@@
 	(label "D0"
 		(at 105.41 151.13 0)
-		(fields_autoplaced yes)
 		(effects
 			(font
@@
 	(label "D2"
 		(at 179.07 74.93 0)
-		(fields_autoplaced yes)
 		(effects
 			(font
@@
 	(label "A0"
 		(at 179.07 57.15 0)
-		(fields_autoplaced yes)
 		(effects
 			(font
@@
 	(label "D5"
 		(at 105.41 163.83 0)
-		(fields_autoplaced yes)
 		(effects
 			(font
@@
 	(label "D5"
 		(at 179.07 82.55 0)
-		(fields_autoplaced yes)
 		(effects
 			(font
@@
 	(label "A3"
 		(at 179.07 64.77 0)
-		(fields_autoplaced yes)
 		(effects
 			(font
@@
 	(label "A1"
 		(at 83.82 176.53 0)
-		(fields_autoplaced yes)
 		(effects
 			(font
@@
 	(label "A2"
 		(at 93.98 62.23 0)
-		(fields_autoplaced yes)
 		(effects
 			(font
@@
 	(label "D7"
 		(at 179.07 87.63 0)
-		(fields_autoplaced yes)
 		(effects
 			(font
@@
 	(label "D0"
 		(at 93.98 69.85 0)
-		(fields_autoplaced yes)
 		(effects
 			(font
@@
 	(label "D3"
 		(at 93.98 77.47 0)
-		(fields_autoplaced yes)
 		(effects
 			(font
@@
 	(label "D1"
 		(at 105.41 153.67 0)
-		(fields_autoplaced yes)
 		(effects
 			(font
@@
 	(label "D4"
 		(at 105.41 161.29 0)
-		(fields_autoplaced yes)
 		(effects
 			(font
@@
 	(label "D4"
 		(at 93.98 80.01 0)
-		(fields_autoplaced yes)
 		(effects
 			(font
@@
 	(label "D7"
 		(at 93.98 87.63 0)
-		(fields_autoplaced yes)
 		(effects
 			(font
@@
 	(label "A2"
 		(at 179.07 62.23 0)
-		(fields_autoplaced yes)
 		(effects
 			(font
@@
 	(label "D1"
 		(at 179.07 72.39 0)
-		(fields_autoplaced yes)
 		(effects
 			(font
@@
 	(label "D2"
 		(at 93.98 74.93 0)
-		(fields_autoplaced yes)
 		(effects
 			(font
@@
 	(label "D6"
 		(at 179.07 85.09 0)
-		(fields_autoplaced yes)
 		(effects
 			(font
@@
 	(label "D2"
 		(at 105.41 156.21 0)
-		(fields_autoplaced yes)
 		(effects
 			(font
@@
 		(shape output)
 		(at 71.12 74.93 180)
-		(fields_autoplaced yes)
 		(effects
 			(font
@@
 		(shape input)
 		(at 200.66 17.78 180)
-		(fields_autoplaced yes)
 		(effects
 			(font
@@
 		(shape input)
 		(at 72.39 77.47 180)
-		(fields_autoplaced yes)
 		(effects
 			(font
@@
 		(shape output)
 		(at 71.12 80.01 180)
-		(fields_autoplaced yes)
 		(effects
 			(font
@@
 		(shape input)
 		(at 200.66 25.4 180)
-		(fields_autoplaced yes)
 		(effects
 			(font
@@
 		(shape input)
 		(at 172.72 17.78 180)
-		(fields_autoplaced yes)
 		(effects
 			(font
@@
 		(shape bidirectional)
 		(at 172.72 20.32 180)
-		(fields_autoplaced yes)
 		(effects
 			(font
@@
 		(shape input)
 		(at 74.93 146.05 180)
-		(fields_autoplaced yes)
 		(effects
 			(font
@@
 		(shape input)
 		(at 73.66 82.55 180)
-		(fields_autoplaced yes)
 		(effects
 			(font
@@
 		(shape input)
 		(at 185.42 110.49 0)
-		(fields_autoplaced yes)
 		(effects
 			(font
@@
 		(shape input)
 		(at 97.79 110.49 0)
-		(fields_autoplaced yes)
 		(effects
 			(font
@@
 			)
 		)
-		(property "Footprint" ""
+		(property "Footprint" "Capacitor_THT:CP_Radial_D4.0mm_P1.50mm"
 			(at 239.7252 25.4 0)
 			(effects
@@
 			)
 		)
-		(property "Footprint" ""
+		(property "Footprint" "Capacitor_THT:CP_Radial_D4.0mm_P1.50mm"
 			(at 230.8352 25.4 0)
 			(effects
@@
 			)
 		)
-		(property "Footprint" ""
+		(property "Footprint" "Capacitor_THT:CP_Radial_D4.0mm_P1.50mm"
 			(at 220.6752 25.4 0)
 			(effects
@@
 			)
 		)
-		(property "Footprint" ""
+		(property "Footprint" "Capacitor_THT:CP_Radial_D4.0mm_P1.50mm"
 			(at 209.2452 25.4 0)
 			(effects
