File: schematics/io-2.kicad_sch (KiCad schematic)
At the start: 14 parts, among them J2 FDC Connector, J3 IDE Connector, U11 WD1772, U4 74LS574, U5 74LS245, U6 74LS245, U7 74LS574

Commit message: Small tweaks here and there. Added a lot of missing footprint definitions.
Parts:
- C3, C4, C5, C6, C7: footprint (none) -> Capacitor_THT:CP_Radial_D4.0mm_P1.50mm
- D2: footprint (none) -> LED_THT:LED_D3.0mm
- R5: footprint Resistor_THT:R_Axial_DIN0411_L9.9mm_D3.6mm_P12.70mm_Horizontal -> Resistor_SMD:R_0805_2012Metric_Pad1.20x1.40mm_HandSolder
